File: Julia Pro 400 Eagle Daughter Board/JP Eagle Daughter Board.brd (EAGLE design)
At the start: 110.2 x 84.7 mm, 43 parts, among them J13 M_DET, J3 SERVO, J4 24V, J5 Z_OUT, J8 CF, K3 FFC/FPC/34PIN/1MMPITCH/TOPLOCK, X1 AUTO BED LEVEL - NANO, X10 AUTO BED LEVEL - RP2040, X11 Z_LIM, X12 Y_LIM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

Commit message: Update
Parts:
- removed U$3: MAKEININDIA, FracktalWorks_Eagle_Library:MAKEININDIA
- moved X3 0.76 mm to (104.6, 20.8)
Routing:
- net 24V: track 99.2 -> 101.4 mm
- net BT0: track 14.0 -> 13.3 mm
Other:
- board text added: "A0+"
- board text added: "A0-"
- board text added: "A1+"
- board text added: "A1-"
- board text added: "B0+"
- board text added: "B0-"
- board text added: "B1+"
- board text added: "B1-"
