File: Julia Pro 400 Eagle Daughter Board/JP Eagle Daughter Board.sch (EAGLE design)
At the start: 42 parts, among them J13 M_DET, J3 SERVO, J4 24V, J5 Z_OUT, J8 CF, K3 FFC/FPC/34PIN/1MMPITCH/TOPLOCK, X1 AUTO BED LEVEL - NANO, X10 AUTO BED LEVEL - RP2040, X11 Z_LIM, X12 Y_LIM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

Commit message: Update
Parts:
- removed U$3: MAKEININDIA, FracktalWorks_Eagle_Library:MAKEININDIA
Changed lines of the file:
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@@
 <part name="J13" library="SparkFun-Connectors" deviceset="CONN_03" device="" value="M_DET"/>
 <part name="X10" library="Rembrandt Electronics - JST XH Connectors v1-0" deviceset="JST-XH-03-PIN" device="-LONG-PAD" value="AUTO BED LEVEL - RP2040"/>
-<part name="U$3" library="FracktalWorks_Eagle_Library" deviceset="MAKEININDIA" device=""/>
 <part name="X12" library="Rembrandt Electronics - JST XH Connectors v1-0" deviceset="JST-XH-02-PIN" device="-LONG-PAD" value="Y_LIM"/>
 <part name="K3" library="FracktalWorks_Eagle_Library" deviceset="FFC/FPC/34PIN/1MMPITCH/TOPLOCK" device=""/>
@@
 <attribute name="NAME" x="246.38" y="189.738" size="1.524" layer="95"/>
 </instance>
-<instance part="U$3" gate="G$1" x="281.94" y="223.52" smashed="yes"/>
 <instance part="X12" gate="-2" x="240.03" y="71.12" smashed="yes">
 <attribute name="NAME" x="242.57" y="70.358" size="1.524" layer="95"/>
